Commit message: added motor speed limits to the robot description

File: config/URDF/robot.urdf.xacro (robot description, xacro)
@@ -9,9 +9,12 @@
         base_joint_min="${base_joint_min}"
         base_joint_max="${base_joint_max}"
+        base_joint_max_speed="${base_joint_max_speed}"
         shoulder_joint_min="${shoulder_joint_min}"
         shoulder_joint_max="${shoulder_joint_max}"
+        shoulder_joint_max_speed="${shoulder_joint_max_speed}"
         elbow_joint_min="${elbow_joint_min}"
         elbow_joint_max="${elbow_joint_max}"
         elbow_joint_offset="${elbow_joint_offset}"
+        elbow_joint_max_speed="${elbow_joint_max_speed}"
     />
     <link name = "gnd_base_link">

File: config/URDF/robot_variables.xacro (robot description, xacro)
@@ -8,9 +8,12 @@
 	<xacro:property name="base_joint_max" value="1.3962634015954636"/>
 	<xacro:property name="base_joint_offset" value="0.0"/>
+	<xacro:property name="base_joint_max_speed" value="2.0943951023931953"/>
 	<xacro:property name="shoulder_joint_min" value="-1.5707963267948966"/>
 	<xacro:property name="shoulder_joint_max" value="1.361356816555577"/>
 	<xacro:property name="shoulder_joint_offset" value="0.0"/>
+	<xacro:property name="shoulder_joint_max_speed" value="2.8902652413026098"/>
 	<xacro:property name="elbow_joint_min" value="-2.6179938779914944"/>
 	<xacro:property name="elbow_joint_max" value="2.076941809873252"/>
 	<xacro:property name="elbow_joint_offset" value="0.04"/>
+	<xacro:property name="elbow_joint_max_speed" value="1.2566370614359172"/>
 </robot>
